File: test_projects/kicad9/test_project.kicad_pcb (KiCad board)
At the start: 8 copper layers, 57.6 x 50 mm, 91 parts, among them J1 HDMI_A, J2 Conn_01x02_Pin, J3 Barrel_Jack_MountingPin, J4 Conn_01x35_Pin, U1 ASDMB-xxxMHz, U2 ADV7611, U3 LM3880, U4 AP2112K-1.8, U6 RT9742AGJ5F

Commit message: [#91282] Update test projects
Routing:
- added copper zone on F.Cu, net (none)
