File: test_projects/kicad9/test_project.kicad_sch (KiCad schematic)
At the start: 3 parts

Commit message: [#91282] Update test projects
Changed lines of the file:
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@@
+		)
+	)
+	(text_box "aaaaa"
+		(exclude_from_sim yes)
+		(at 13.97 81.28 90)
+		(size 38.1 35.56)
+		(margins 0.9525 0.9525 0.9525 0.9525)
+		(stroke
+			(width 0.0254)
+			(type dash)
+			(color 132 0 132 1)
+		)
+		(fill
+			(type color)
+			(color 0 255 0 0.9)
+		)
+		(effects
+			(font
+				(size 1.2954 1.2954)
+				(color 132 0 0 1)
+			)
+			(justify right)
+			(href "https://google.com")
 		)
 	)
@@
 			(at 368.3 220.98 0)
 			(effects
-				(hide yes)
-			)
-			(effects
-				(font
-					(size 1.27 1.27)
-				)
+				(font
+					(size 1.27 1.27)
+				)
+				(hide yes)
 			)
 		)
@@
 			(at 368.3 220.98 0)
 			(effects
-				(hide yes)
-			)
-			(effects
-				(font
-					(size 1.27 1.27)
-				)
+				(font
+					(size 1.27 1.27)
+				)
+				(hide yes)
 			)
 		)
@@
 			(at 368.3 220.98 0)
 			(effects
-				(hide yes)
-			)
-			(effects
-				(font
-					(size 1.27 1.27)
-				)
+				(font
+					(size 1.27 1.27)
+				)
+				(hide yes)
 			)
 		)
@@
 			(at 368.3 226.06 0)
 			(effects
-				(hide yes)
-			)
-			(effects
-				(font
-					(size 1.27 1.27)
-				)
+				(font
+					(size 1.27 1.27)
+				)
+				(hide yes)
 			)
 		)
@@
 			(at 368.3 226.06 0)
 			(effects
-				(hide yes)
-			)
-			(effects
-				(font
-					(size 1.27 1.27)
-				)
+				(font
+					(size 1.27 1.27)
+				)
+				(hide yes)
 			)
 		)
@@
 			(at 368.3 226.06 0)
 			(effects
-				(hide yes)
-			)
-			(effects
-				(font
-					(size 1.27 1.27)
-				)
+				(font
+					(size 1.27 1.27)
+				)
+				(hide yes)
 			)
 		)
@@
 			(at 368.3 231.14 0)
 			(effects
-				(hide yes)
-			)
-			(effects
-				(font
-					(size 1.27 1.27)
-				)
+				(font
+					(size 1.27 1.27)
+				)
+				(hide yes)
 			)
 		)
@@
 			(at 368.3 231.14 0)
 			(effects
-				(hide yes)
-			)
-			(effects
-				(font
-					(size 1.27 1.27)
-				)
+				(font
+					(size 1.27 1.27)
+				)
+				(hide yes)
 			)
 		)
@@
 			(at 368.3 231.14 0)
 			(effects
-				(hide yes)
-			)
-			(effects
-				(font
-					(size 1.27 1.27)
-				)
+				(font
+					(size 1.27 1.27)
+				)
+				(hide yes)
 			)
 		)
@@
 			(at 39.37 254 0)
 			(effects
-				(hide yes)
-			)
-			(effects
-				(font
-					(size 1.27 1.27)
-				)
+				(font
+					(size 1.27 1.27)
+				)
+				(hide yes)
 			)
 		)
@@
 			(at 39.37 276.86 0)
 			(effects
-				(hide yes)
-			)
-			(effects
-				(font
-					(size 1.27 1.27)
-				)
+				(font
+					(size 1.27 1.27)
+				)
+				(hide yes)
 			)
 		)
@@
 			(at 39.37 266.7 0)
 			(effects
-				(hide yes)
-			)
-			(effects
-				(font
-					(size 1.27 1.27)
-				)
+				(font
+					(size 1.27 1.27)
+				)
+				(hide yes)
 			)
 		)
@@
 			(at 39.37 266.7 0)
 			(effects
-				(hide yes)
-			)
-			(effects
-				(font
-					(size 1.27 1.27)
-				)
+				(font
+					(size 1.27 1.27)
+				)
+				(hide yes)
 			)
 		)
@@
 			(at 39.37 266.7 0)
 			(effects
-				(hide yes)
-			)
-			(effects
-				(font
-					(size 1.27 1.27)
-				)
+				(font
+					(size 1.27 1.27)
+				)
+				(hide yes)
 			)
 		)
@@
 			(at 365.76 246.38 0)
 			(effects
-				(hide yes)
-			)
-			(effects
-				(font
-					(size 1.27 1.27)
-				)
+				(font
+					(size 1.27 1.27)
+				)
+				(hide yes)
 			)
 		)
@@
 			(at 365.76 240.03 0)
 			(effects
-				(hide yes)
-			)
-			(effects
-				(font
-					(size 1.27 1.27)
-				)
+				(font
+					(size 1.27 1.27)
+				)
+				(hide yes)
 			)
 		)
@@
 			(at 365.76 240.03 0)
 			(effects
-				(hide yes)
-			)
-			(effects
-				(font
-					(size 1.27 1.27)
-				)
+				(font
+					(size 1.27 1.27)
+				)
+				(hide yes)
 			)
 		)
@@
 			(at 365.76 240.03 0)
 			(effects
-				(hide yes)
-			)
-			(effects
-				(font
-					(size 1.27 1.27)
-				)
+				(font
+					(size 1.27 1.27)
+				)
+				(hide yes)
 			)
 		)
@@
 		)
 		(fill
-			(color 0 0 0 0)
+			(color 0 0 0 0.0000)
 		)
 		(property "Sheetname" "Receiver"
@@
 		)
 		(fill
-			(color 0 0 0 0)
+			(color 0 0 0 0.0000)
 		)
 		(property "Sheetname" "Connectors"
@@
 		)
 		(fill
-			(color 0 0 0 0)
+			(color 0 0 0 0.0000)
 		)
 		(property "Sheetname" "multi-channel-test"
@@
 		)
 		(fill
-			(color 0 0 0 0)
+			(color 0 0 0 0.0000)
 		)
 		(property "Sheetname" "Power"
@@
 		)
 		(fill
-			(color 0 0 0 0)
+			(color 0 0 0 0.0000)
 		)
 		(property "Sheetname" "multi-channel-test1"
